File: 02 board-schematic/ESP32_monitor_sp/board.brd (EAGLE design)
At the start: 100 x 70 mm, 33 parts, among them IC1 ESP32-WROOM-32D__4MB_PS_, IC4 LM1117IMP-3.3_NOPB

Commit message: Update Board
Parts:
- moved T1 15.2 mm to (39.7, 58.5)
- moved IC3 15.0 mm to (39.8, 50.9)
- flipped C5 to the bottom
- flipped C6 to the bottom
Connections:
- removed net IO13: IC1.16, JP4.29
- removed net N$1: JP3.1, U$1.SD_SCK
- removed net N$2: JP3.2, U$1.SD_MISO
- removed net N$3: JP3.3, U$1.SD_MOSI
- removed net N$4: JP3.4, U$1.SD_CS
- new net SD_CS: IC1.16, JP3.4, JP4.29, U$1.SD_CS
- net TFT_CLK: now also JP3.1, U$1.SD_SCK
- net TFT_MISO: now also JP3.2, U$1.SD_MISO
- net TFT_MOSI: now also JP3.3, U$1.SD_MOSI
Routing:
- net SD_CS: track 0.00 -> 91.7 mm
- net TFT_MOSI: track 74.9 -> 154.0 mm, vias 3 -> 1
- net TFT_CLK: track 78.1 -> 140.4 mm, vias 0 -> 4
- net 3V3: track 236.8 -> 289.4 mm, vias 2 -> 4
- net TFT_MISO: track 91.7 -> 142.0 mm, vias 0 -> 2
- net TFT_CS: track 65.2 -> 107.2 mm, vias 3 -> 0
- net UART2_MCU2MP3: track 88.2 -> 58.1 mm, vias 2 -> 3
- net EN: track 123.2 -> 152.1 mm, vias 3 -> 4
- net GND: track 297.2 -> 274.6 mm, vias 4 -> 91
- net TFT_LED: track 95.4 -> 76.6 mm, vias 3 -> 0
- net D+: track 19.0 -> 34.7 mm
- net D-: track 24.9 -> 39.5 mm
- net IO13: track 13.1 -> 0.00 mm
- net IO0: track 150.2 -> 138.9 mm, vias 5 -> 3
- net TOUCH_CS: track 35.2 -> 46.1 mm, vias 3 -> 2
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Other:
- board text added: "BOOT"
- board text added: "EN"
- board text added: "ESP32_Monitor_R2"
- board text removed: "ESP32_Monitor"
