File: 02 board-schematic/ESP32_monitor_sp/board.sch (EAGLE design)
At the start: 33 parts, among them IC1 ESP32-WROOM-32D__4MB_PS_, IC4 LM1117IMP-3.3_NOPB

Commit message: Update Board
Connections:
- removed net IO13: IC1.IO13, JP4.29
- removed net N$1: JP3.1, U$1.SD_SCK
- removed net N$2: JP3.2, U$1.SD_MISO
- removed net N$3: JP3.3, U$1.SD_MOSI
- removed net N$4: JP3.4, U$1.SD_CS
- new net SD_CS: IC1.IO13, JP3.4, JP4.29, U$1.SD_CS
- net TFT_CLK: now also JP3.1, U$1.SD_SCK
- net TFT_MISO: now also JP3.2, U$1.SD_MISO
- net TFT_MOSI: now also JP3.3, U$1.SD_MOSI
